File: Peak_Control_HAT_RevA/Peak_Control_HAT_RevA.kicad_sch (KiCad schematic)
At the start: 10 parts, among them J2 24V_IN, U1 TPS272C45C_RHF24, U2 TPS272C45C_RHF24

Commit message: Changed placeholder items with TPS272C45C
Parts:
- U1, U2: footprint (none) -> Peak_Control_HAT:VQFN-24_5x4mm_P0.5mm_EP; symbol Connector_Generic:Conn_02x12_Odd_Even -> Peak_Control_HAT:TPS272C45C
Changed lines of the file:
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@@
 	)
 	(symbol
-		(lib_id "Connector_Generic:Conn_02x12_Odd_Even")
+		(lib_id "Peak_Control_HAT:TPS272C45C")
 		(at 175.26 39.37 0)
 		(unit 1)
@@
 			)
 		)
-		(property "Footprint" ""
+		(property "Footprint" "Peak_Control_HAT:VQFN-24_5x4mm_P0.5mm_EP"
 			(at 175.26 39.37 0)
-			(show_name no)
-			(do_not_autoplace no)
-			(effects
-				(font
-					(size 1.27 1.27)
-				)
-			)
-		)
-		(property "Datasheet" ""
+			(hide yes)
+			(show_name no)
+			(do_not_autoplace no)
+			(effects
+				(font
+					(size 1.27 1.27)
+				)
+			)
+		)
+		(property "Datasheet" "https://www.ti.com/lit/ds/symlink/tps272c45.pdf"
 			(at 175.26 39.37 0)
-			(show_name no)
-			(do_not_autoplace no)
-			(effects
-				(font
-					(size 1.27 1.27)
-				)
-			)
-		)
-		(property "Description" ""
+			(hide yes)
+			(show_name no)
+			(do_not_autoplace no)
+			(effects
+				(font
+					(size 1.27 1.27)
+				)
+			)
+		)
+		(property "Description" "Dual-channel 36V industrial smart high-side switch with current sense and diagnostics, C variant"
 			(at 175.26 39.37 0)
+			(hide yes)
 			(show_name no)
 			(do_not_autoplace no)
@@
 		)
 		(pin "21"
+		)
+		(pin "25"
 		)
 		(instances
@@
 	)
 	(symbol
-		(lib_id "Connector_Generic:Conn_02x12_Odd_Even")
+		(lib_id "Peak_Control_HAT:TPS272C45C")
 		(at 175.26 125.73 0)
 		(unit 1)
@@
 			)
 		)
-		(property "Footprint" ""
+		(property "Footprint" "Peak_Control_HAT:VQFN-24_5x4mm_P0.5mm_EP"
 			(at 175.26 125.73 0)
-			(show_name no)
-			(do_not_autoplace no)
-			(effects
-				(font
-					(size 1.27 1.27)
-				)
-			)
-		)
-		(property "Datasheet" ""
+			(hide yes)
+			(show_name no)
+			(do_not_autoplace no)
+			(effects
+				(font
+					(size 1.27 1.27)
+				)
+			)
+		)
+		(property "Datasheet" "https://www.ti.com/lit/ds/symlink/tps272c45.pdf"
 			(at 175.26 125.73 0)
-			(show_name no)
-			(do_not_autoplace no)
-			(effects
-				(font
-					(size 1.27 1.27)
-				)
-			)
-		)
-		(property "Description" ""
+			(hide yes)
+			(show_name no)
+			(do_not_autoplace no)
+			(effects
+				(font
+					(size 1.27 1.27)
+				)
+			)
+		)
+		(property "Description" "Dual-channel 36V industrial smart high-side switch with current sense and diagnostics, C variant"
 			(at 175.26 125.73 0)
+			(hide yes)
 			(show_name no)
 			(do_not_autoplace no)
@@
 		(pin "24"
 		)
+		(pin "25"
+		)
 		(instances

Commit message: Added U1 connections with ERC report
Parts:
- added C3: 1uF, symbol Device:C
- added R1.1, R1.2: 13.7k 1%, symbol Device:R
- added R1.3, R1.4: 100K, symbol Device:R
- added R1.5: 10K, symbol Device:R
- added R1.6: 2.4K, symbol Device:R
Connections:
- net +24V_FIELD: now also U1.23 (VS), U1.24 (VS), U1.8 (VS), U1.9 (VS)
- net FIELD_GND: now also U1.14 (LATCH), U1.17 (GND), U1.18 (ILIMD), U1.25 (EP_GND), C3.2, R1.1.2, R1.2.2, R1.3.1, R1.4.1, R1.6.1
- net OUT1_24V: now reaches U1.1 (OUT1)
- net OUT1_24V: now also U1.2 (OUT1), U1.3 (OUT1)
- net GPIO20: now reaches U1.10 (~{FLT})
- net GPIO20: now also R1.5.2
- net ADC_U1_SNS: now reaches U1.11 (SNS)
- net ADC_U1_SNS: now also R1.6.2
- net 3.3V: now reaches U1.12 (DIA_EN)
- net 3.3V: now also R1.5.1
- net GPIO5: now reaches U1.13 (SEL)
- net GPIO19: now reaches U1.15 (EN2)
- net GPIO19: now also R1.3.2
- net GPIO16: now reaches U1.16 (EN1)
- net GPIO16: now also R1.4.2
- net VDD_NODE: now reaches U1.19 (VDD)
- net VDD_NODE: now also C3.1
- net at U1.20 (ILIM2): now also R1.1.1
- net at U1.21 (ILIM1): now also R1.2.1
- net OUT2_24V: now reaches U1.5 (OUT2)
- net OUT2_24V: now also U1.6 (OUT2), U1.7 (OUT2)

Commit message: Updated U1 connections and ERC report
Parts:
- removed C3: 1uF, symbol Device:C
- removed R11: 13.7k 1% ILIM1 (~1.5A nominal), symbol Device:R
- removed R12: 13.7k 1% ILIM2 (~1.5A nominal), symbol Device:R
- removed R13: 499R 1% SNS, symbol Device:R
Connections:
- net VDD_NODE is gone; now on net FIELD_GND: U1.19 (VDD)
