File: Peak_Control_SSR_Interface_RevA/Peak_Control_SSR_Interface_RevA.kicad_pcb (KiCad board)
At the start: 4 copper layers, 115 x 70 mm, 26 parts, among them J1 Pi/Control GPIO Conn., J2 24V_IN, J3 PROJECTOR_SW24V_GND, J4 VIEWER_SW24V_GND, J5 AUX1_SW24V_GND, J6 AUX2_SW24V_GND, U1 G3VM-61GR2, U2 G3VM-61GR2, U3 G3VM-61GR2, U4 G3VM-61GR2

Commit message: Checkpoint for completed RevA, requires final verification
Parts:
- added REF**: MountingHole_2.7mm_M2.5, MountingHole:MountingHole_2.7mm_M2.5, F.Cu at (5.50, 60.0)
- added REF**: MountingHole_2.7mm_M2.5, MountingHole:MountingHole_2.7mm_M2.5, F.Cu at (5.50, 11.0)
- added REF**: MountingHole_2.7mm_M2.5, MountingHole:MountingHole_2.7mm_M2.5, F.Cu at (63.5, 60.0)
- added REF**: MountingHole_2.7mm_M2.5, MountingHole:MountingHole_2.7mm_M2.5, F.Cu at (63.5, 11.0)
- moved J1 37.2 mm to (49.7, 7.50), turned to 180 degrees
- moved R17 10.0 mm to (65.0, 19.5), turned to -90 degrees
- moved R16 9.71 mm to (65.0, 34.5), turned to -90 degrees
- moved R18 9.62 mm to (65.0, 4.50), turned to -90 degrees
- moved R13 9.55 mm to (69.0, 17.5)
- moved R14 9.19 mm to (69.0, 2.50)
- moved D1 9.01 mm to (33.0, 55.0), turned to -90 degrees
- moved U1 8.92 mm to (70.2, 50.9), turned to -90 degrees
- moved R12 8.90 mm to (69.0, 32.5)
- moved U2 8.60 mm to (70.3, 35.9), turned to -90 degrees
- moved U3 8.24 mm to (70.3, 20.9), turned to -90 degrees
- moved U4 7.89 mm to (70.3, 5.92), turned to -90 degrees
- moved R11 7.34 mm to (68.9, 47.5), turned to 180 degrees
- moved R15 5.65 mm to (64.9, 49.5), turned to -90 degrees
- moved C2 3.35 mm to (47.5, 52.5), turned to -90 degrees
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Connections:
- J1 pad 1: /PI_GND -> /GPIO_IN4
- J1 pad 2: /GPIO_IN1 -> /GPIO_IN3
- J1 pad 4: /GPIO_IN3 -> /GPIO_IN1
- J1 pad 5: /GPIO_IN4 -> /PI_GND
Routing:
- net /GPIO_IN4: track 64.9 -> 21.1 mm
- net /GPIO_IN3: track 71.5 -> 29.5 mm
- net /+24V_FIELD: track 153.0 -> 131.7 mm
- net /GPIO_IN2: track 55.9 -> 41.0 mm
- net /GPIO_IN1: track 65.4 -> 58.5 mm
- net /PI_GND: track 44.8 -> 40.3 mm, vias 4 -> 5
- net /FIELD_GND: track 46.1 -> 48.2 mm
- net Net-(R13-Pad1): track 2.61 -> 3.54 mm
- net Net-(R14-Pad1): track 2.61 -> 3.54 mm
- net Net-(R12-Pad1): track 2.76 -> 3.54 mm
- added copper zone on In2.Cu, net /FIELD_GND
- added copper zone on In2.Cu, net /PI_GND
- removed copper zone on In1.Cu, net /FIELD_GND
- removed copper zone on In1.Cu, net /PI_GND
Other:
- board size 115 x 70 mm -> 98 x 70 mm
- board text added: "+ Out1 -"
- board text added: "+ Out2 -"
- board text added: "+ Out3 -"
- board text added: "+ Out4 -"
- board text added: "In4 In3 In2 In1 Gnd"
- board text added: "MC INPUT 3.3V ONLY"
- board text added: "PEAK CONTROL SSR INTERFACE"
- board text removed: "PEAK CONTROL HAT - SSR"

Commit message: Minor text updates before final pre-fab review
Other:
- board text added: "REV A1.1"
- board text removed: "REV A1-DRAFT / G3VM-61GR2"
Changed lines of the file:
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@@
 	(paper "A4")
 	(title_block
-		(title "Peak Control HAT SSR Rev A - Mechanical / Placement Skeleton")
-		(date "2026-08-27")
-		(rev "A1-DRAFT")
+		(title "Peak Control SSR Interface Rev A1.1")
+		(date "2026-09-01")
+		(rev "A1.1")
 		(company "Peak Projections")
+		(comment 1 "Mechanical / Placement Skeleton")
 	)
 	(layers
@@
 		)
 	)
-	(gr_text "REV A1-DRAFT / G3VM-61GR2"
-		(at 7.5 27.5 270)
+	(gr_text "REV A1.1"
+		(at 8.5 19 270)
 		(layer "F.SilkS")
 		(effects

Commit message: Replaced fuseholder F1 footprint
Parts:
- F1: footprint Fuse:Fuseholder_Clip-5x20mm_Bel_FC-203-22_Lateral_P17.80x5.00mm_D1.17mm_Horizontal -> JLC:FUSE-TH_L22.6-W9.0
- moved F1 6.62 mm to (33.5, 65.0)
Routing:
- net Net-(J2-Pin_1): track 12.0 -> 8.21 mm
- net /+24V_FIELD: track 131.7 -> 129.5 mm

Commit message: Changed terminal block footprints to production items
Parts:
- J1: footprint TerminalBlock_Phoenix:TerminalBlock_Phoenix_MKDS-1,5-5-5.08_1x05_P5.08mm_Horizontal -> JLC:CONN-TH_5P-P5.08_DIBO_DB128V-5.08-5P-GN-S
- J2, J3, J4, J5, J6: footprint TerminalBlock_Phoenix:TerminalBlock_Phoenix_MKDS-1,5-2-5.08_1x02_P5.08mm_Horizontal -> JLC:CONN-TH_YC0220500000G
- moved J1 10.2 mm to (39.4, 7.50)
- moved J4 2.62 mm to (84.0, 37.0)
- moved J3 2.58 mm to (84.0, 52.0)
- moved J6 2.58 mm to (84.0, 7.00)
- moved J2 2.55 mm to (54.5, 63.2)
- moved J5 2.50 mm to (84.0, 22.5)
Routing:
- net /GPIO_IN4: track 21.1 -> 23.0 mm
