File: Peak_Control_SSR_Interface_RevA/Peak_Control_SSR_Interface_RevA.kicad_sch (KiCad schematic)
At the start: 26 parts, among them J1 Pi/Control GPIO Conn., J2 24V_IN, J3 PROJECTOR_SW24V_GND, J4 VIEWER_SW24V_GND, J5 AUX1_SW24V_GND, J6 AUX2_SW24V_GND, U1 G3VM-61GR2, U2 G3VM-61GR2, U3 G3VM-61GR2, U4 G3VM-61GR2

Commit message: Checkpoint for completed RevA, requires final verification
Connections:
- net GPIO_IN1: now also J1.4 (Pin_4); no longer J1.2 (Pin_2)
- net GPIO_IN3: now also J1.2 (Pin_2); no longer J1.4 (Pin_4)
- net GPIO_IN4: now also J1.1 (Pin_1); no longer J1.5 (Pin_5)
- net PI_GND: now also J1.5 (Pin_5); no longer J1.1 (Pin_1)
Changed lines of the file:
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@@
 	)
 	(label "GPIO_IN3"
-		(at 236.22 41.91 0)
+		(at 236.22 36.83 0)
 		(effects
 			(font
@@
 	)
 	(label "PI_GND"
-		(at 236.22 34.29 0)
+		(at 236.22 44.45 0)
 		(effects
 			(font
@@
 	)
 	(label "GPIO_IN4"
-		(at 236.22 44.45 0)
+		(at 236.22 34.29 0)
 		(effects
 			(font
@@
 	)
 	(label "GPIO_IN1"
-		(at 236.22 36.83 0)
-		(effects
-			(font
+		(at 236.22 41.91 0)
+		(effects
+			(font

Commit message: Minor text updates before final pre-fab review
Other:
- note added: "Move SSR Resistor Networks to Board Center, Provide Jumpers For 3.3v/5v Selection"
- title: Peak Control SSR Interface Rev A - Power Output Core -> Peak Control SSR Interface Rev A1.1 - Power Output Core
Changed lines of the file:
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@@
 	(paper "A4")
 	(title_block
-		(title "Peak Control SSR Interface Rev A - Power Output Core")
+		(title "Peak Control SSR Interface Rev A1.1 - Power Output Core")
 		(date "2026-08-27")
 		(rev "A1-DRAFT")
@@
 		(exclude_from_sim no)
 		(at 19.05 63.5 0)
+		(effects
+			(font
+				(size 1.397 1.397)
+			)
+			(justify left bottom)
+		)
+	)
+	(text "5V Regulator from 24V Supply - Can provide fan supply or power for MC/Pi (need 6A for Pi)"
+		(exclude_from_sim no)
+		(at 37.338 159.004 0)
 		(effects
 			(font
@@
 		)
 	)
-	(text "5V Regulator from 24V Supply - Can provide fan supply or power for MC/Pi (need 6A for Pi)"
+	(text "Move SSR Resistor Networks to Board Center, Provide Jumpers For 3.3v/5v Selection "
 		(exclude_from_sim no)
 		(at 37.338 155.194 0)

Commit message: Additional minor text updates before final pre-fab review
Other:
- note added: "NOTES FOR FUTURE REVISIONS"
- note removed: "RETAINED FUNCTIONS / NEXT SHEET WORK"
Changed lines of the file:
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@@
 	(title_block
 		(title "Peak Control SSR Interface Rev A1.1 - Power Output Core")
-		(date "2026-08-27")
-		(rev "A1-DRAFT")
+		(date "2026-09-01")
+		(rev "A1.1")
 		(company "Peak Projections")
 		(comment 1 "24V input protection + 4x isolated Omron G3VM-61GR2 outputs")
 	)
-	(text "RETAINED FUNCTIONS / NEXT SHEET WORK"
+	(text "NOTES FOR FUTURE REVISIONS"
 		(exclude_from_sim no)
-		(at 34.798 147.574 0)
+		(at 36.322 159.004 0)
 		(effects
 			(font
@@
 	(text "5V Regulator from 24V Supply - Can provide fan supply or power for MC/Pi (need 6A for Pi)"
 		(exclude_from_sim no)
-		(at 37.338 159.004 0)
+		(at 37.084 168.656 0)
 		(effects
 			(font
@@
 	(text "Move SSR Resistor Networks to Board Center, Provide Jumpers For 3.3v/5v Selection "
 		(exclude_from_sim no)
-		(at 37.338 155.194 0)
+		(at 37.084 164.846 0)
 		(effects
 			(font

Commit message: Replaced fuseholder F1 footprint
Parts:
- C1: MPN (none) -> 50RX3047MT78X11.5; Manufacturer (none) -> Rubycon; Supplier (none) -> JLCPCB/LCSC; Supplier PN (none) -> C473223
- C2: MPN (none) -> 08055C105K4T2A; Manufacturer (none) -> Kyocera AVX; Supplier (none) -> JLCPCB/LCSC; Supplier PN (none) -> C779994
- D1: MPN (none) -> SMBJ33A; Manufacturer (none) -> Zhengxin; Supplier (none) -> JLCPCB/LCSC; Supplier PN (none) -> C5261717
- D11, D12, D13, D14: MPN (none) -> 1N4007; Manufacturer (none) -> ST(Semtech); Supplier (none) -> JLCPCB/LCSC; Supplier PN (none) -> C106903
- F1: footprint Fuse:Fuseholder_Clip-5x20mm_Bel_FC-203-22_Lateral_P17.80x5.00mm_D1.17mm_Horizontal -> JLC:FUSE-TH_L22.6-W9.0; MPN (none) -> 5x20 BLX-A XC-7; Manufacturer (none) -> Xucheng Elec; Supplier (none) -> JLCPCB/LCSC; Supplier PN (none) -> C3131
- J1: MPN (none) -> DB128V-5.08-5P-GN-S; Manufacturer (none) -> Dorabo; Supplier (none) -> JLCPCB/LCSC; Supplier PN (none) -> C2927513
- J2, J3, J4, J5, J6: MPN (none) -> YC0220500000G; Manufacturer (none) -> Amphenol ICC; Supplier (none) -> JLCPCB/LCSC; Supplier PN (none) -> C2683165
- R11, R12, R13, R14: MPN (none) -> RC0805FR-07390RL; Manufacturer (none) -> Yageo; Supplier (none) -> JLCPCB/LCSC; Supplier PN (none) -> C114543
- R15, R16, R17, R18: MPN (none) -> RC0805FR-07100KL; Manufacturer (none) -> Yageo; Supplier (none) -> JLCPCB/LCSC; Supplier PN (none) -> C96346
- U1, U2, U3, U4: MPN (none) -> G3VM-61GR2(TR05); Manufacturer (none) -> Omron; Supplier (none) -> JLCPCB/LCSC; Supplier PN (none) -> C2653911

Commit message: Changed terminal block footprints to production items
Parts:
- J1: footprint TerminalBlock_Phoenix:TerminalBlock_Phoenix_MKDS-1,5-5-5.08_1x05_P5.08mm_Horizontal -> JLC:CONN-TH_5P-P5.08_DIBO_DB128V-5.08-5P-GN-S
- J2, J3, J4, J5, J6: footprint TerminalBlock_Phoenix:TerminalBlock_Phoenix_MKDS-1,5-2-5.08_1x02_P5.08mm_Horizontal -> JLC:CONN-TH_YC0220500000G
Changed lines of the file:
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@@
 			)
 		)
-		(property "Footprint" "TerminalBlock_Phoenix:TerminalBlock_Phoenix_MKDS-1,5-2-5.08_1x02_P5.08mm_Horizontal"
+		(property "Footprint" "JLC:CONN-TH_YC0220500000G"
 			(at 30.48 27.94 0)
 			(hide yes)
@@
 			)
 		)
-		(property "Footprint" "TerminalBlock_Phoenix:TerminalBlock_Phoenix_MKDS-1,5-2-5.08_1x02_P5.08mm_Horizontal"
+		(property "Footprint" "JLC:CONN-TH_YC0220500000G"
 			(at 120.65 86.36 0)
 			(hide yes)
@@
 			)
 		)
-		(property "Footprint" "TerminalBlock_Phoenix:TerminalBlock_Phoenix_MKDS-1,5-2-5.08_1x02_P5.08mm_Horizontal"
+		(property "Footprint" "JLC:CONN-TH_YC0220500000G"
 			(at 255.27 96.52 0)
 			(hide yes)
@@
 			)
 		)
-		(property "Footprint" "TerminalBlock_Phoenix:TerminalBlock_Phoenix_MKDS-1,5-2-5.08_1x02_P5.08mm_Horizontal"
+		(property "Footprint" "JLC:CONN-TH_YC0220500000G"
 			(at 123.19 121.92 0)
 			(hide yes)
@@
 			)
 		)
-		(property "Footprint" "TerminalBlock_Phoenix:TerminalBlock_Phoenix_MKDS-1,5-2-5.08_1x02_P5.08mm_Horizontal"
+		(property "Footprint" "JLC:CONN-TH_YC0220500000G"
 			(at 255.27 130.81 0)
 			(hide yes)
@@
 			)
 		)
-		(property "Footprint" "TerminalBlock_Phoenix:TerminalBlock_Phoenix_MKDS-1,5-5-5.08_1x05_P5.08mm_Horizontal"
+		(property "Footprint" "JLC:CONN-TH_5P-P5.08_DIBO_DB128V-5.08-5P-GN-S"
 			(at 255.27 39.37 0)
 			(hide yes)
