File: Peak_Control_2CH_SSR_Interface_RevA/Peak_Control_2CH_SSR_Interface_RevA.kicad_sch (KiCad schematic)
At the start: 16 parts, among them J1 Pi/Control GPIO Conn., J2 24V_IN, J3 PROJECTOR_SW24V_GND, J4 VIEWER_SW24V_GND, U1 G3VM-61GR2, U2 G3VM-61GR2

Commit message: Pre-fab checkpoint for 2ch version, file cleanup
Parts:
- J1: MPN DB128V-5.08-5P-GN-S -> DB128V-5.08-3P-GN-S; Supplier PN C2927513 -> C2915640
Changed lines of the file:
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@@
 			)
 		)
-		(property "MPN" "DB128V-5.08-5P-GN-S"
+		(property "MPN" "DB128V-5.08-3P-GN-S"
 			(at 255.27 39.37 0)
 			(hide yes)
@@
 			)
 		)
-		(property "Supplier PN" "C2927513"
+		(property "Supplier PN" "C2915640"
 			(at 255.27 39.37 0)
 			(hide yes)
